File: DWM Breakout.brd (EAGLE design)
At the start: 33.2 x 33.3 mm, 3 parts, among them U1 DWM1000

Commit message: Add files via upload
Parts:
- removed U1: DWM1000, DWM1000:DWM1000
- added B1: ARDUINO_PRO_MINI, SparkFun-Boards:ARDUINO_PRO_MINI
- added LSP1, LSP2: SE14, solpad:SE14
- added R1: (no value), rcl:0207/10
- added SV3: (no value), con-lstb:MA04-1
Connections:
- removed net N$1: SV1.1, U1.1
- removed net N$10: SV1.10, U1.10
- removed net N$11: SV1.11, U1.11
- removed net N$12: SV1.12, U1.12
- removed net N$13: SV2.3, U1.15
- removed net N$14: SV2.1, U1.13
- removed net N$15: SV2.2, U1.14
- removed net N$16: SV2.4, U1.16
- removed net N$17: SV2.5, U1.17
- removed net N$18: SV2.6, U1.18
- removed net N$19: SV2.7, U1.19
- removed net N$20: SV2.8, U1.20
- removed net N$21: SV2.9, U1.21
- removed net N$22: SV2.10, U1.22
- removed net N$23: SV2.11, U1.23
- removed net N$25: SV2.12, U1.24
- removed net N$9: SV1.9, U1.9
- new net 3V3: B1.21, LSP1.MP, SV1.5, SV1.6, SV1.7
- new net GND: B1.23, B1.4, LSP2.MP, R1.1, SV1.8, SV2.11, SV2.12, SV2.9, SV3.1
- new net IRQ: B1.5, R1.2, SV2.10
- new net RAW: B1.24
- new net RST: B1.12, SV1.3
- net N$2: now also B1.15, SV2.7; no longer SV1.2, U1.2
- net N$3: now also B1.1, SV3.4; no longer SV1.3, U1.3
- net N$4: now also B1.16, SV2.8; no longer SV1.4, U1.4
- net N$5: now also B1.14, SV2.6; no longer SV1.5, U1.5
- net N$6: now also B1.13, SV2.5; no longer SV1.6, U1.6
- net N$7: now also B1.2, SV3.3; no longer SV1.7, U1.7
- net N$8: now also B1.3, SV3.2; no longer SV1.8, U1.8
Routing:
- net GND: track 0.00 -> 118.4 mm, vias 0 -> 2
- net 3V3: track 0.00 -> 50.1 mm, vias 0 -> 1
- net RST: track 0.00 -> 27.1 mm, vias 0 -> 1
- net N$14: track 25.0 -> 0.00 mm
- net N$12: track 25.0 -> 0.00 mm
- net IRQ: track 0.00 -> 24.7 mm, vias 0 -> 1
- net N$15: track 21.7 -> 0.00 mm
- net N$11: track 21.7 -> 0.00 mm
- net N$10: track 18.6 -> 0.00 mm
- net N$13: track 18.6 -> 0.00 mm
- net N$8: track 14.3 -> 32.1 mm
- net N$16: track 15.3 -> 0.00 mm
- net N$9: track 15.3 -> 0.00 mm
- net N$17: track 14.3 -> 0.00 mm
- net N$18: track 13.8 -> 0.00 mm
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- added copper zone on layer 1, net GND
- added copper zone on layer 16, net GND
Other:
- board size 33.2 x 33.3 mm -> 39.4 x 37 mm
- board text added: "05/03/2019"
- board text added: "Alaa Al Ahmar Amera Johar Zahra Zaghloul"
- board text removed: "DWM1000 Breakout Board"
