File: DWM Breakout.sch (EAGLE design)
At the start: 3 parts, among them U1 DWM1000

Commit message: Add files via upload
Parts:
- removed U1: DWM1000, DWM1000:DWM1000
- added B1: ARDUINO_PRO_MINI, SparkFun-Boards:ARDUINO_PRO_MINI
- added LSP1, LSP2: SE14, solpad:SE14
- added R1: (no value), rcl:R-EU_0207/10
- added SV3: (no value), con-lstb:MA04-1
Connections:
- removed net N$1: SV1.1, U1.EXTON
- removed net N$10: SV1.10, U1.GPIO5/SPIPOL
- removed net N$11: SV1.11, U1.GPIO4
- removed net N$12: SV1.12, U1.GPIO3/TXLED
- removed net N$13: SV2.3, U1.GPIO0/RXOKLED
- removed net N$14: SV2.1, U1.GPIO2/RXLED
- removed net N$15: SV2.2, U1.GPIO1/SFDLED
- removed net N$16: SV2.4, U1.VSS@5
- removed net N$17: SV2.5, U1.!SPICS
- removed net N$18: SV2.6, U1.SPIMOSI
- removed net N$19: SV2.7, U1.SPIMISO
- removed net N$20: SV2.8, U1.SPICLK
- removed net N$21: SV2.9, U1.VSS@4
- removed net N$22: SV2.10, U1.IRQ/GPIO8
- removed net N$23: SV2.11, U1.VSS@3
- removed net N$25: SV2.12, U1.VSS@2
- removed net N$9: SV1.9, U1.GPIO6
- new net 3V3: B1.VCC, LSP1.MP, SV1.5, SV1.6, SV1.7
- new net GND: B1.GND, B1.GND@2, LSP2.MP, R1.1, SV1.8, SV2.11, SV2.12, SV2.9, SV3.1
- new net IRQ: B1.2, R1.2, SV2.10
- new net RST: B1.*9, SV1.3
- net N$2: now also B1.12, SV2.7; no longer SV1.2, U1.WAKEUP
- net N$3: now also B1.TXO, SV3.4; no longer SV1.3, U1.!RST
- net N$4: now also B1.13, SV2.8; no longer SV1.4, U1.GPIO7
- net N$5: now also B1.*11, SV2.6; no longer SV1.5, U1.VDDAON
- net N$6: now also B1.*10, SV2.5; no longer SV1.6, U1.VDD@2
- net N$7: now also B1.RXI, SV3.3; no longer SV1.7, U1.VDD
- net N$8: now also B1.RST, SV3.2; no longer SV1.8, U1.VSS
Other:
- moved on the sheet: SV1, SV2
